Commit message: missing tf broadcasting added and turned on odom publisher

File: fastbot_description/models/urdf/fastbot_OG.urdf (robot description, URDF)
Before this commit: robot fastbot, 7 links, 6 joints
Links:
- removed link fastbot_base_link
- removed link fastbot_camera
- removed link fastbot_motor_1
- removed link fastbot_motor_2
- removed link fastbot_wheel_left
- removed link fastbot_wheel_right
- added link base_link, mass 0.24695; collision mesh filename=package://fastbot_description/onshape/assets/fastbot_chassi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; visual mesh filename=package://fastbot_description/onshape/assets/fastbot_chassi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
- added link camera, mass 1e-09; collision mesh filename=package://fastbot_description/onshape/assets/part_33.stl; visual mesh filename=package://fastbot_description/onshape/assets/part_33.stl
- added link motor, mass 0.0339689; collision mesh filename=package://fastbot_description/onshape/assets/fastbot_motor.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; visual mesh filename=package://fastbot_description/onshape/assets/fastbot_motor.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
- added link motor_2, mass 0.0339689; collision mesh filename=package://fastbot_description/onshape/assets/fastbot_motor.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; visual mesh filename=package://fastbot_description/onshape/assets/fastbot_motor.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
- added link wheel_left, mass 1e-09; collision mesh filename=package://fastbot_description/onshape/assets/wheel_d65x25_v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; collision mesh filename=package://fastbot_description/onshape/assets/wheel_d65x25_v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
- added link wheel_right, mass 1e-09; collision mesh filename=package://fastbot_description/onshape/assets/wheel_d65x25_v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; collision mesh filename=package://fastbot_description/onshape/assets/wheel_d65x25_v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
Joints:
- removed joint fastbot_camera
- added joint camera: type fixed, parent base_link, child camera, origin xyz=0.0105 -0.0668336 0.09765 rpy=-1.5708 1.14468e-45 6.41848e-15, axis 0 0 1, limit effort=10 velocity=10
- joint left_motor: child fastbot_motor_2 -> motor_2; parent fastbot_base_link -> base_link
- joint left_wheel: child fastbot_wheel_left -> wheel_left; parent fastbot_motor_2 -> motor_2
- joint lidar: parent fastbot_base_link -> base_link
- joint right_motor: child fastbot_motor_1 -> motor; parent fastbot_base_link -> base_link
- joint right_wheel: child fastbot_wheel_right -> wheel_right; parent fastbot_motor_1 -> motor
